File: Hardware/SparkFun_Pro_Micro.sch (EAGLE design)
At the start: 33 parts, among them U2 MIC5219, U3 ATMEGA32U4, Y1 16MHz

Commit message: Swap USB-B micro with USB-A male connector
Parts:
- removed X1: (no value), Testing:USB-ABIN&OUT
- added J1: USB-A-H, SparkFun-Connectors:USB-A-H
Connections:
- removed net N$8: R5.2, X1.D+
- new net N$9: J1.D+, R5.2
- net GND: now also J1.GND; no longer X1.GND
- net N$6: now also J1.D-; no longer X1.D-
- net UVCC: now also J1.VBUS; no longer X1.VBUS
Other:
- moved on the sheet: R5, R7
Changed lines of the file:
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@@
 <?xml version="1.0" encoding="utf-8"?>
 <!DOCTYPE eagle SYSTEM "eagle.dtd">
-<eagle version="7.3.0">
+<eagle version="7.7.0">
 <drawing>
 <settings>
@@
 <part name="R5" library="SparkFun" deviceset="RESISTOR" device="0603-RES" value="22"/>
 <part name="R7" library="SparkFun" deviceset="RESISTOR" device="0603-RES" value="22"/>
-<part name="X1" library="Testing" deviceset="USB-AB" device="IN&amp;OUT"/>
 <part name="GND3" library="SparkFun" deviceset="GND" device=""/>
 <part name="JP1" library="SparkFun" deviceset="FIDUCIAL" device="UFIDUCIAL"/>
@@
 <part name="P+1" library="SparkFun" deviceset="VCC" device=""/>
 <part name="P+2" library="SparkFun" deviceset="VCC" device=""/>
+<part name="J1" library="SparkFun-Connectors" deviceset="USB" device="-A-H"/>
 </parts>
 <sheets>
@@
 <attribute name="VALUE" x="207.137" y="68.326" size="1.778" layer="96" rot="R270"/>
 </instance>
-<instance part="R5" gate="G$1" x="121.92" y="88.9" smashed="yes" rot="R180">
-<attribute name="NAME" x="117.856" y="90.678" size="1.778" layer="95"/>
+<instance part="R5" gate="G$1" x="121.92" y="81.28" smashed="yes" rot="R180">
+<attribute name="NAME" x="117.856" y="83.058" size="1.778" layer="95"/>
+<attribute name="VALUE" x="123.19" y="83.058" size="1.778" layer="96"/>
+</instance>
+<instance part="R7" gate="G$1" x="121.92" y="88.9" smashed="yes" rot="R180">
+<attribute name="NAME" x="118.11" y="90.678" size="1.778" layer="95"/>
 <attribute name="VALUE" x="123.19" y="90.678" size="1.778" layer="96"/>
 </instance>
-<instance part="R7" gate="G$1" x="121.92" y="81.28" smashed="yes" rot="R180">
-<attribute name="NAME" x="118.11" y="83.058" size="1.778" layer="95"/>
-<attribute name="VALUE" x="123.19" y="83.058" size="1.778" layer="96"/>
-</instance>
-<instance part="X1" gate="G$1" x="101.6" y="86.36" rot="MR0"/>
 <instance part="GND3" gate="1" x="109.22" y="73.66"/>
 <instance part="JP1" gate="G$1" x="238.76" y="38.1"/>
@@
 <instance part="P+1" gate="1" x="200.66" y="60.96" rot="R180"/>
 <instance part="P+2" gate="1" x="210.82" y="60.96" rot="R180"/>
+<instance part="J1" gate="G$1" x="104.14" y="91.44" rot="R180"/>
 </instances>
 <busses>
@@
 <wire x1="106.68" y1="91.44" x2="109.22" y2="91.44" width="0.1524" layer="91"/>
 <wire x1="109.22" y1="91.44" x2="109.22" y2="76.2" width="0.1524" layer="91"/>
-<pinref part="X1" gate="G$1" pin="GND"/>
 <pinref part="GND3" gate="1" pin="GND"/>
+<pinref part="J1" gate="G$1" pin="GND"/>
 </segment>
 <segment>
@@
 </segment>
 <segment>
-<wire x1="106.68" y1="81.28" x2="111.76" y2="81.28" width="0.1524" layer="91"/>
-<wire x1="111.76" y1="81.28" x2="111.76" y2="76.2" width="0.1524" layer="91"/>
 <wire x1="111.76" y1="76.2" x2="132.08" y2="76.2" width="0.1524" layer="91"/>
 <label x="129.54" y="76.2" size="1.778" layer="95"/>
-<pinref part="X1" gate="G$1" pin="VBUS"/>
+<pinref part="J1" gate="G$1" pin="VBUS"/>
+<wire x1="106.68" y1="88.9" x2="111.76" y2="88.9" width="0.1524" layer="91"/>
+<wire x1="111.76" y1="88.9" x2="111.76" y2="76.2" width="0.1524" layer="91"/>
 </segment>
 <segment>
@@
 </segment>
 <segment>
-<wire x1="127" y1="81.28" x2="132.08" y2="81.28" width="0.1524" layer="91"/>
-<label x="129.54" y="81.28" size="1.778" layer="95"/>
+<wire x1="127" y1="88.9" x2="132.08" y2="88.9" width="0.1524" layer="91"/>
+<label x="129.54" y="88.9" size="1.778" layer="95"/>
 <pinref part="R7" gate="G$1" pin="1"/>
 </segment>
@@
 </segment>
 <segment>
-<wire x1="127" y1="88.9" x2="132.08" y2="88.9" width="0.1524" layer="91"/>
-<label x="129.54" y="88.9" size="1.778" layer="95"/>
+<wire x1="127" y1="81.28" x2="132.08" y2="81.28" width="0.1524" layer="91"/>
+<label x="129.54" y="81.28" size="1.778" layer="95"/>
 <pinref part="R5" gate="G$1" pin="1"/>
 </segment>
@@
 <net name="N$6" class="0">
 <segment>
-<wire x1="106.68" y1="83.82" x2="114.3" y2="83.82" width="0.1524" layer="91"/>
-<wire x1="114.3" y1="83.82" x2="114.3" y2="81.28" width="0.1524" layer="91"/>
-<wire x1="114.3" y1="81.28" x2="116.84" y2="81.28" width="0.1524" layer="91"/>
-<pinref part="R7" gate="G$1" pin="2"/>
-<pinref part="X1" gate="G$1" pin="D-"/>
-</segment>
-</net>
-<net name="N$8" class="0">
-<segment>
-<wire x1="106.68" y1="86.36" x2="114.3" y2="86.36" width="0.1524" layer="91"/>
 <wire x1="114.3" y1="86.36" x2="114.3" y2="88.9" width="0.1524" layer="91"/>
 <wire x1="114.3" y1="88.9" x2="116.84" y2="88.9" width="0.1524" layer="91"/>
-<pinref part="R5" gate="G$1" pin="2"/>
-<pinref part="X1" gate="G$1" pin="D+"/>
+<pinref part="R7" gate="G$1" pin="2"/>
+<pinref part="J1" gate="G$1" pin="D-"/>
+<wire x1="106.68" y1="86.36" x2="114.3" y2="86.36" width="0.1524" layer="91"/>
 </segment>
 </net>
@@
 </segment>
 </net>
+<net name="N$9" class="0">
+<segment>
+<pinref part="J1" gate="G$1" pin="D+"/>
+<wire x1="106.68" y1="83.82" x2="114.3" y2="83.82" width="0.1524" layer="91"/>
+<wire x1="114.3" y1="83.82" x2="114.3" y2="81.28" width="0.1524" layer="91"/>
+<pinref part="R5" gate="G$1" pin="2"/>
+<wire x1="114.3" y1="81.28" x2="116.84" y2="81.28" width="0.1524" layer="91"/>
+</segment>
+</net>
